File: KiCad/DoubleRow6SlotBackplane/DoubleRow6SlotBackplane.kicad_pcb (KiCad board)
At the start: 2 copper layers, 16 parts, among them J0 Conn_02x20_Row_Letter_First, J1 Conn_02x20_Row_Letter_First, J10 Conn_02x20_Row_Letter_First, J11 Conn_02x20_Row_Letter_First, J12 Conn_02x20_Row_Letter_First, J13 Conn_02x20_Row_Letter_First, J14 Conn_02x20_Row_Letter_First, J15 Conn_02x20_Row_Letter_First, J2 Conn_02x20_Row_Letter_First, J3 Conn_02x20_Row_Letter_First, J4 Conn_02x20_Row_Letter_First, J5 Conn_02x20_Row_Letter_First, J6 Conn_02x20_Row_Letter_First, J7 Conn_02x20_Row_Letter_First, J8 Conn_02x20_Row_Letter_First, J9 Conn_02x20_Row_Letter_First

Commit message: Adding 6 slot backplane files
Parts:
- removed J14, J15: Conn_02x20_Row_Letter_First, Connector_PinHeader_2.54mm:PinHeader_2x20_P2.54mm_Horizontal
- added P0: Conn_02x20_Row_Letter_First, Connector_PinHeader_2.54mm:PinHeader_2x20_P2.54mm_Horizontal, F.Cu at (203.2, 40.6)
- added P1: Conn_02x20_Row_Letter_First, Connector_PinHeader_2.54mm:PinHeader_2x20_P2.54mm_Horizontal, F.Cu at (203.2, 101.6)
- added REF**: MountingHole_3.2mm_M3_Pad, MountingHole:MountingHole_3.2mm_M3_Pad, F.Cu at (76.2, 43.2)
- added REF**: MountingHole_3.2mm_M3_Pad, MountingHole:MountingHole_3.2mm_M3_Pad, F.Cu at (195.6, 147.3)
- added REF**: MountingHole_3.2mm_M3_Pad, MountingHole:MountingHole_3.2mm_M3_Pad, F.Cu at (76.2, 147.3)
- added REF**: MountingHole_3.2mm_M3_Pad, MountingHole:MountingHole_3.2mm_M3_Pad, F.Cu at (195.6, 43.2)
- moved J13 82.4 mm to (188.0, 101.6)
- moved J11 80.7 mm to (167.6, 101.6)
- moved J9 79.5 mm to (147.3, 101.6)
- moved J7 78.6 mm to (127.0, 101.6)
- moved J3 78.3 mm to (86.4, 101.6)
- moved J5 78.2 mm to (106.7, 101.6)
- moved J1 75.5 mm to (68.6, 101.6)
- moved J0 65.7 mm to (68.6, 40.6)
- moved J12 37.5 mm to (188.0, 40.6)
- moved J10 32.2 mm to (167.6, 40.6)
- moved J8 27.3 mm to (147.3, 40.6)
- moved J6 23.0 mm to (127.0, 40.6)
- moved J4 19.5 mm to (106.7, 40.6)
- moved J2 17.5 mm to (86.4, 40.6)
Connections:
- J0 pad 1: /~{SYSRST} -> /5V
- J0 pad 11: /D3 -> /D2
- J0 pad 13: /D4 -> /D3
- J0 pad 15: /D5 -> /D4
- J0 pad 17: /D6 -> /D5
- J0 pad 19: /D7 -> /D6
- J0 pad 2: /C0 -> /GND
- J0 pad 21: /A0 -> /D7
- J0 pad 23: /A1 -> /A0
- J0 pad 25: /A2 -> /A1
- J0 pad 27: /A3 -> /A2
- J0 pad 29: /A4 -> /A3
- J0 pad 3: /SYSCLK -> /~{SYSRST}
- J0 pad 31: /A5 -> /A4
- J0 pad 33: /A6 -> /A5
- J0 pad 35: /A7 -> /A6
- J0 pad 37: GND -> /A7
- J0 pad 38: GND -> /C18
- J0 pad 39: /5V -> /C0
- J0 pad 40: /5V -> /C19
- J0 pad 5: /D0 -> /SYSCLK
- J0 pad 7: /D1 -> /D0
- J0 pad 9: /D2 -> /D1
- J1 pad 1: /5V -> /C20
- J1 pad 10: /U8 -> /U13
- J1 pad 11: /C21 -> /OP1
- J1 pad 12: /U9 -> /U14
- J1 pad 13: /C22 -> /OP2
- J1 pad 14: /U10 -> /U15
- J1 pad 15: /C23 -> /OP3
- J1 pad 16: /U11 -> /U16
- J1 pad 17: /OP0 -> /OP4
- J1 pad 18: /U12 -> /U17
- J1 pad 19: /OP1 -> /U0
- J1 pad 2: /5V -> /U9
- J1 pad 20: /U13 -> /U18
- J1 pad 21: /OP2 -> /U1
- J1 pad 22: /U14 -> /U19
- J1 pad 23: /OP3 -> /U2
- J1 pad 24: /U15 -> /U20
- J1 pad 25: /OP4 -> /U3
- J1 pad 26: /U16 -> /U21
- J1 pad 27: /U0 -> /U4
- J1 pad 28: /U17 -> /U22
- J1 pad 29: /U1 -> /U5
- J1 pad 3: GND -> /C21
- J1 pad 30: /U18 -> /U23
- J1 pad 31: /U2 -> /U6
- J1 pad 32: /U19 -> /U24
- J1 pad 33: /U3 -> /U7
- J1 pad 34: /U20 -> /U25
- J1 pad 35: /U4 -> /U8
- J1 pad 36: /U21 -> /U26
- J1 pad 37: /U5 -> /IE0
- J1 pad 38: /U22 -> /IE0
- J1 pad 39: /IE0 -> /5V
- J1 pad 4: GND -> /U10
- J1 pad 40: /IE0 -> /GND
- J1 pad 5: /C18 -> /C22
- J1 pad 6: /U6 -> /U11
- J1 pad 7: /C19 -> /C23
- J1 pad 8: /U7 -> /U12
- J1 pad 9: /C20 -> /OP0
- J10 pad 1: /~{SYSRST} -> /5V
- J10 pad 11: /D3 -> /D2
- J10 pad 13: /D4 -> /D3
- J10 pad 15: /D5 -> /D4
- J10 pad 17: /D6 -> /D5
- J10 pad 19: /D7 -> /D6
- J10 pad 2: /C0 -> /GND
- J10 pad 21: /A0 -> /D7
- J10 pad 23: /A1 -> /A0
- J10 pad 25: /A2 -> /A1
- J10 pad 27: /A3 -> /A2
- J10 pad 29: /A4 -> /A3
- J10 pad 3: /SYSCLK -> /~{SYSRST}
- J10 pad 31: /A5 -> /A4
- J10 pad 33: /A6 -> /A5
- J10 pad 35: /A7 -> /A6
- J10 pad 37: GND -> /A7
- J10 pad 38: GND -> /C18
- J10 pad 39: /5V -> /C0
- J10 pad 40: /5V -> /C19
- J10 pad 5: /D0 -> /SYSCLK
- J10 pad 7: /D1 -> /D0
- J10 pad 9: /D2 -> /D1
- J11 pad 1: /5V -> /C20
- J11 pad 10: /U8 -> /U13
- J11 pad 11: /C21 -> /OP1
- J11 pad 12: /U9 -> /U14
- J11 pad 13: /C22 -> /OP2
- J11 pad 14: /U10 -> /U15
- J11 pad 15: /C23 -> /OP3
- J11 pad 16: /U11 -> /U16
- J11 pad 17: /OP0 -> /OP4
- J11 pad 18: /U12 -> /U17
- J11 pad 19: /OP1 -> /U0
- J11 pad 2: /5V -> /U9
- J11 pad 20: /U13 -> /U18
- J11 pad 21: /OP2 -> /U1
- J11 pad 22: /U14 -> /U19
- J11 pad 23: /OP3 -> /U2
- J11 pad 24: /U15 -> /U20
- J11 pad 25: /OP4 -> /U3
- J11 pad 26: /U16 -> /U21
- J11 pad 27: /U0 -> /U4
- J11 pad 28: /U17 -> /U22
- J11 pad 29: /U1 -> /U5
- J11 pad 3: GND -> /C21
- J11 pad 30: /U18 -> /U23
- J11 pad 31: /U2 -> /U6
- J11 pad 32: /U19 -> /U24
- J11 pad 33: /U3 -> /U7
- J11 pad 34: /U20 -> /U25
- J11 pad 35: /U4 -> /U8
- J11 pad 36: /U21 -> /U26
- J11 pad 37: /U5 -> /IE0
- J11 pad 38: /U22 -> /IE0
- J11 pad 39: /IE0 -> /5V
- J11 pad 4: GND -> /U10
- J11 pad 40: /IE0 -> /GND
- J11 pad 5: /C18 -> /C22
- J11 pad 6: /U6 -> /U11
- J11 pad 7: /C19 -> /C23
- J11 pad 8: /U7 -> /U12
- J11 pad 9: /C20 -> /OP0
- J12 pad 1: /~{SYSRST} -> /5V
- J12 pad 11: /D3 -> /D2
- J12 pad 13: /D4 -> /D3
- J12 pad 15: /D5 -> /D4
- J12 pad 17: /D6 -> /D5
- J12 pad 19: /D7 -> /D6
- J12 pad 2: /C0 -> /GND
- J12 pad 21: /A0 -> /D7
- J12 pad 23: /A1 -> /A0
- J12 pad 25: /A2 -> /A1
- J12 pad 27: /A3 -> /A2
- J12 pad 29: /A4 -> /A3
- J12 pad 3: /SYSCLK -> /~{SYSRST}
- J12 pad 31: /A5 -> /A4
- J12 pad 33: /A6 -> /A5
- J12 pad 35: /A7 -> /A6
- J12 pad 37: GND -> /A7
- J12 pad 38: GND -> /C18
- J12 pad 39: /5V -> /C0
- J12 pad 40: /5V -> /C19
- J12 pad 5: /D0 -> /SYSCLK
- J12 pad 7: /D1 -> /D0
- J12 pad 9: /D2 -> /D1
- J13 pad 1: /5V -> /C20
- J13 pad 10: /U8 -> /U13
- J13 pad 11: /C21 -> /OP1
- J13 pad 12: /U9 -> /U14
- J13 pad 13: /C22 -> /OP2
- J13 pad 14: /U10 -> /U15
- J13 pad 15: /C23 -> /OP3
- J13 pad 16: /U11 -> /U16
- J13 pad 17: /OP0 -> /OP4
- J13 pad 18: /U12 -> /U17
- J13 pad 19: /OP1 -> /U0
- J13 pad 2: /5V -> /U9
- J13 pad 20: /U13 -> /U18
- J13 pad 21: /OP2 -> /U1
- J13 pad 22: /U14 -> /U19
- J13 pad 23: /OP3 -> /U2
- J13 pad 24: /U15 -> /U20
- J13 pad 25: /OP4 -> /U3
- J13 pad 26: /U16 -> /U21
- J13 pad 27: /U0 -> /U4
- J13 pad 28: /U17 -> /U22
- J13 pad 29: /U1 -> /U5
- J13 pad 3: GND -> /C21
- J13 pad 30: /U18 -> /U23
- J13 pad 31: /U2 -> /U6
- J13 pad 32: /U19 -> /U24
- J13 pad 33: /U3 -> /U7
- J13 pad 34: /U20 -> /U25
- J13 pad 35: /U4 -> /U8
- J13 pad 36: /U21 -> /U26
- J13 pad 37: /U5 -> /IE0
- J13 pad 38: /U22 -> /IE0
- J13 pad 39: /IE0 -> /5V
- J13 pad 4: GND -> /U10
- J13 pad 40: /IE0 -> /GND
- J13 pad 5: /C18 -> /C22
- J13 pad 6: /U6 -> /U11
- J13 pad 7: /C19 -> /C23
- J13 pad 8: /U7 -> /U12
- J13 pad 9: /C20 -> /OP0
- J2 pad 1: /~{SYSRST} -> /5V
- J2 pad 11: /D3 -> /D2
- J2 pad 13: /D4 -> /D3
- J2 pad 15: /D5 -> /D4
- J2 pad 17: /D6 -> /D5
- J2 pad 19: /D7 -> /D6
- J2 pad 2: /C0 -> /GND
- J2 pad 21: /A0 -> /D7
- J2 pad 23: /A1 -> /A0
- J2 pad 25: /A2 -> /A1
- J2 pad 27: /A3 -> /A2
- J2 pad 29: /A4 -> /A3
- J2 pad 3: /SYSCLK -> /~{SYSRST}
- J2 pad 31: /A5 -> /A4
- J2 pad 33: /A6 -> /A5
- J2 pad 35: /A7 -> /A6
- J2 pad 37: GND -> /A7
- J2 pad 38: GND -> /C18
- J2 pad 39: /5V -> /C0
- J2 pad 40: /5V -> /C19
- J2 pad 5: /D0 -> /SYSCLK
- J2 pad 7: /D1 -> /D0
- J2 pad 9: /D2 -> /D1
- J3 pad 1: /5V -> /C20
- J3 pad 10: /U8 -> /U13
- J3 pad 11: /C21 -> /OP1
- J3 pad 12: /U9 -> /U14
- J3 pad 13: /C22 -> /OP2
- J3 pad 14: /U10 -> /U15
- J3 pad 15: /C23 -> /OP3
- J3 pad 16: /U11 -> /U16
- J3 pad 17: /OP0 -> /OP4
- J3 pad 18: /U12 -> /U17
- J3 pad 19: /OP1 -> /U0
- J3 pad 2: /5V -> /U9
- J3 pad 20: /U13 -> /U18
- J3 pad 21: /OP2 -> /U1
- J3 pad 22: /U14 -> /U19
- J3 pad 23: /OP3 -> /U2
- J3 pad 24: /U15 -> /U20
- J3 pad 25: /OP4 -> /U3
- J3 pad 26: /U16 -> /U21
- J3 pad 27: /U0 -> /U4
- J3 pad 28: /U17 -> /U22
- J3 pad 29: /U1 -> /U5
- J3 pad 3: GND -> /C21
- J3 pad 30: /U18 -> /U23
- J3 pad 31: /U2 -> /U6
- J3 pad 32: /U19 -> /U24
- J3 pad 33: /U3 -> /U7
- J3 pad 34: /U20 -> /U25
- J3 pad 35: /U4 -> /U8
- J3 pad 36: /U21 -> /U26
- J3 pad 37: /U5 -> /IE0
- J3 pad 38: /U22 -> /IE0
- J3 pad 39: /IE0 -> /5V
- J3 pad 4: GND -> /U10
- J3 pad 40: /IE0 -> /GND
- J3 pad 5: /C18 -> /C22
- J3 pad 6: /U6 -> /U11
- J3 pad 7: /C19 -> /C23
- J3 pad 8: /U7 -> /U12
- J3 pad 9: /C20 -> /OP0
- J4 pad 1: /~{SYSRST} -> /5V
- J4 pad 11: /D3 -> /D2
- J4 pad 13: /D4 -> /D3
- J4 pad 15: /D5 -> /D4
- J4 pad 17: /D6 -> /D5
- J4 pad 19: /D7 -> /D6
- J4 pad 2: /C0 -> /GND
- J4 pad 21: /A0 -> /D7
- J4 pad 23: /A1 -> /A0
- J4 pad 25: /A2 -> /A1
- J4 pad 27: /A3 -> /A2
- J4 pad 29: /A4 -> /A3
- J4 pad 3: /SYSCLK -> /~{SYSRST}
- J4 pad 31: /A5 -> /A4
- J4 pad 33: /A6 -> /A5
- J4 pad 35: /A7 -> /A6
- J4 pad 37: GND -> /A7
- J4 pad 38: GND -> /C18
- J4 pad 39: /5V -> /C0
- J4 pad 40: /5V -> /C19
- J4 pad 5: /D0 -> /SYSCLK
- J4 pad 7: /D1 -> /D0
- J4 pad 9: /D2 -> /D1
- J5 pad 1: /5V -> /C20
- J5 pad 10: /U8 -> /U13
- J5 pad 11: /C21 -> /OP1
- J5 pad 12: /U9 -> /U14
- J5 pad 13: /C22 -> /OP2
- J5 pad 14: /U10 -> /U15
- J5 pad 15: /C23 -> /OP3
- J5 pad 16: /U11 -> /U16
- J5 pad 17: /OP0 -> /OP4
- J5 pad 18: /U12 -> /U17
- J5 pad 19: /OP1 -> /U0
- J5 pad 2: /5V -> /U9
- J5 pad 20: /U13 -> /U18
- J5 pad 21: /OP2 -> /U1
- J5 pad 22: /U14 -> /U19
- J5 pad 23: /OP3 -> /U2
- J5 pad 24: /U15 -> /U20
- J5 pad 25: /OP4 -> /U3
- J5 pad 26: /U16 -> /U21
- J5 pad 27: /U0 -> /U4
- J5 pad 28: /U17 -> /U22
- J5 pad 29: /U1 -> /U5
- J5 pad 3: GND -> /C21
- J5 pad 30: /U18 -> /U23
- J5 pad 31: /U2 -> /U6
- J5 pad 32: /U19 -> /U24
- J5 pad 33: /U3 -> /U7
- J5 pad 34: /U20 -> /U25
- J5 pad 35: /U4 -> /U8
- J5 pad 36: /U21 -> /U26
- J5 pad 37: /U5 -> /IE0
- J5 pad 38: /U22 -> /IE0
- J5 pad 39: /IE0 -> /5V
- J5 pad 4: GND -> /U10
- J5 pad 40: /IE0 -> /GND
- J5 pad 5: /C18 -> /C22
- J5 pad 6: /U6 -> /U11
- J5 pad 7: /C19 -> /C23
- J5 pad 8: /U7 -> /U12
- J5 pad 9: /C20 -> /OP0
- J6 pad 1: /~{SYSRST} -> /5V
- J6 pad 11: /D3 -> /D2
- J6 pad 13: /D4 -> /D3
- J6 pad 15: /D5 -> /D4
- J6 pad 17: /D6 -> /D5
- J6 pad 19: /D7 -> /D6
- J6 pad 2: /C0 -> /GND
- J6 pad 21: /A0 -> /D7
- J6 pad 23: /A1 -> /A0
- J6 pad 25: /A2 -> /A1
- J6 pad 27: /A3 -> /A2
- J6 pad 29: /A4 -> /A3
- J6 pad 3: /SYSCLK -> /~{SYSRST}
- J6 pad 31: /A5 -> /A4
- J6 pad 33: /A6 -> /A5
- J6 pad 35: /A7 -> /A6
- J6 pad 37: GND -> /A7
- J6 pad 38: GND -> /C18
- J6 pad 39: /5V -> /C0
- J6 pad 40: /5V -> /C19
- J6 pad 5: /D0 -> /SYSCLK
- J6 pad 7: /D1 -> /D0
- J6 pad 9: /D2 -> /D1
- J7 pad 1: /5V -> /C20
- J7 pad 10: /U8 -> /U13
- J7 pad 11: /C21 -> /OP1
- J7 pad 12: /U9 -> /U14
- J7 pad 13: /C22 -> /OP2
- J7 pad 14: /U10 -> /U15
- J7 pad 15: /C23 -> /OP3
- J7 pad 16: /U11 -> /U16
- J7 pad 17: /OP0 -> /OP4
- J7 pad 18: /U12 -> /U17
- J7 pad 19: /OP1 -> /U0
- J7 pad 2: /5V -> /U9
- J7 pad 20: /U13 -> /U18
- J7 pad 21: /OP2 -> /U1
- J7 pad 22: /U14 -> /U19
- J7 pad 23: /OP3 -> /U2
- J7 pad 24: /U15 -> /U20
- J7 pad 25: /OP4 -> /U3
- J7 pad 26: /U16 -> /U21
- J7 pad 27: /U0 -> /U4
- J7 pad 28: /U17 -> /U22
- J7 pad 29: /U1 -> /U5
- J7 pad 3: GND -> /C21
- J7 pad 30: /U18 -> /U23
- J7 pad 31: /U2 -> /U6
- J7 pad 32: /U19 -> /U24
- J7 pad 33: /U3 -> /U7
- J7 pad 34: /U20 -> /U25
- J7 pad 35: /U4 -> /U8
- J7 pad 36: /U21 -> /U26
- J7 pad 37: /U5 -> /IE0
- J7 pad 38: /U22 -> /IE0
- J7 pad 39: /IE0 -> /5V
- J7 pad 4: GND -> /U10
- J7 pad 40: /IE0 -> /GND
- J7 pad 5: /C18 -> /C22
- J7 pad 6: /U6 -> /U11
- J7 pad 7: /C19 -> /C23
- J7 pad 8: /U7 -> /U12
- J7 pad 9: /C20 -> /OP0
- J8 pad 1: /~{SYSRST} -> /5V
- J8 pad 11: /D3 -> /D2
- J8 pad 13: /D4 -> /D3
- J8 pad 15: /D5 -> /D4
- J8 pad 17: /D6 -> /D5
- J8 pad 19: /D7 -> /D6
- J8 pad 2: /C0 -> /GND
- J8 pad 21: /A0 -> /D7
- J8 pad 23: /A1 -> /A0
- J8 pad 25: /A2 -> /A1
- J8 pad 27: /A3 -> /A2
- J8 pad 29: /A4 -> /A3
- J8 pad 3: /SYSCLK -> /~{SYSRST}
- J8 pad 31: /A5 -> /A4
- J8 pad 33: /A6 -> /A5
- J8 pad 35: /A7 -> /A6
- J8 pad 37: GND -> /A7
- J8 pad 38: GND -> /C18
- J8 pad 39: /5V -> /C0
- J8 pad 40: /5V -> /C19
- J8 pad 5: /D0 -> /SYSCLK
- J8 pad 7: /D1 -> /D0
- J8 pad 9: /D2 -> /D1
- J9 pad 1: /5V -> /C20
- J9 pad 10: /U8 -> /U13
- J9 pad 11: /C21 -> /OP1
- J9 pad 12: /U9 -> /U14
- J9 pad 13: /C22 -> /OP2
- J9 pad 14: /U10 -> /U15
- J9 pad 15: /C23 -> /OP3
- J9 pad 16: /U11 -> /U16
- J9 pad 17: /OP0 -> /OP4
- J9 pad 18: /U12 -> /U17
- J9 pad 19: /OP1 -> /U0
- J9 pad 2: /5V -> /U9
- J9 pad 20: /U13 -> /U18
- J9 pad 21: /OP2 -> /U1
- J9 pad 22: /U14 -> /U19
- J9 pad 23: /OP3 -> /U2
- J9 pad 24: /U15 -> /U20
- J9 pad 25: /OP4 -> /U3
- J9 pad 26: /U16 -> /U21
- J9 pad 27: /U0 -> /U4
- J9 pad 28: /U17 -> /U22
- J9 pad 29: /U1 -> /U5
- J9 pad 3: GND -> /C21
- J9 pad 30: /U18 -> /U23
- J9 pad 31: /U2 -> /U6
- J9 pad 32: /U19 -> /U24
- J9 pad 33: /U3 -> /U7
- J9 pad 34: /U20 -> /U25
- J9 pad 35: /U4 -> /U8
- J9 pad 36: /U21 -> /U26
- J9 pad 37: /U5 -> /IE0
- J9 pad 38: /U22 -> /IE0
- J9 pad 39: /IE0 -> /5V
- J9 pad 4: GND -> /U10
- J9 pad 40: /IE0 -> /GND
- J9 pad 5: /C18 -> /C22
- J9 pad 6: /U6 -> /U11
- J9 pad 7: /C19 -> /C23
- J9 pad 8: /U7 -> /U12
- J9 pad 9: /C20 -> /OP0
Routing:
- net /GND: track 0.00 -> 316.9 mm
- net /5V: track 0.00 -> 304.3 mm
- net /C2: track 0.00 -> 151.2 mm
- net /C1: track 0.00 -> 151.2 mm
- net /C15: track 0.00 -> 147.9 mm
- net /C3: track 0.00 -> 147.9 mm
- net /C17: track 0.00 -> 146.7 mm
- net /U22: track 0.00 -> 146.5 mm
- net /U26: track 0.00 -> 146.5 mm
- net /U25: track 0.00 -> 146.5 mm
- net /U11: track 0.00 -> 146.5 mm
- net /C19: track 0.00 -> 146.5 mm
- net /C12: track 0.00 -> 146.5 mm
- net /U21: track 0.00 -> 146.5 mm
- net /U13: track 0.00 -> 146.5 mm
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Other:
- board outline added: 145.3 x 116.9 mm
- board text added: "+5V"
- board text added: "5V"
- board text added: "A0"
- board text added: "A1"
- board text added: "A2"
- board text added: "A3"
- board text added: "A4"
- board text added: "A5"
- board text added: "A6"
- board text added: "A7"
- board text added: "C0"
- board text added: "C1"
- board text added: "C10"
- board text added: "C11"
- board text added: "C12"
- board text added: "C13"
- board text added: "C14"
- board text added: "C15"
- board text added: "C16"
- board text added: "C17"
- board text added: "C18"
- board text added: "C19"
- board text added: "C2"
- board text added: "C20"
- board text added: "C21"
- board text added: "C22"
- board text added: "C23"
- board text added: "C3"
- board text added: "C4"
- board text added: "C5"
- board text added: "C6"
- board text added: "C7"
- board text added: "C8"
- board text added: "C9"
- board text added: "D0"
- board text added: "D1"
- board text added: "D2"
- board text added: "D3"
- board text added: "D4"
- board text added: "D5"
- board text added: "D6"
- board text added: "D7"
- board text added: "GND"
- board text added: "IE0"
- board text added: "IEI"
- board text added: "OP0"
- board text added: "OP1"
- board text added: "OP2"
- board text added: "OP3"
- board text added: "OP4"
- board text added: "SYSCLK"
- board text added: "U0"
- board text added: "U1"
- board text added: "U10"
- board text added: "U11"
- board text added: "U12"
- board text added: "U13"
- board text added: "U14"
- board text added: "U15"
- board text added: "U16"
- board text added: "U17"
- board text added: "U18"
- board text added: "U19"
- board text added: "U2"
- board text added: "U20"
- board text added: "U21"
- board text added: "U22"
- board text added: "U23"
- board text added: "U24"
- board text added: "U25"
- board text added: "U26"
- board text added: "U3"
- board text added: "U4"
- board text added: "U5"
- board text added: "U6"
- board text added: "U7"
- board text added: "U8"
- board text added: "U9"
- board text added: "~{SYSRST}"
